File: PCB/UFC.kicad_sch (KiCad schematic)
At the start: 101 parts, among them IC0 CD74HCT4067M, IC1 CD74HCT4067M, K0 EP1-3N1S, M0 Fan_3pin, M1 Fan_3pin, M2 Fan_3pin, M3 Fan_3pin, M4 Fan_3pin, M5 Fan_3pin, M6 Fan_3pin, M7 Fan_3pin, Q0 NMOS, Q1 NMOS, Q2 NMOS, Q3 NMOS, Q4 NMOS, Q5 NMOS, Q6 NMOS, Q7 NMOS, Q9 NMOS, SW0 MCU Reset, SW1 Main Power Switch, U0 Pico

Commit message: footprinty dokonczon
w końcu xd
Parts:
- F0: footprint (none) -> Fuse:Fuseholder_Blade_Mini_Keystone_3568
- IC0, IC1: footprint SOIC127P1030X265-24N -> UFC_Lib_FP:SOIC127P1030X265-24N
- K0: footprint EP13N1S -> UFC_Lib_FP:EP13N1S
- R11, R12, R13, R14, R15, R16, R17, R18: footprint (none) -> Resistor_SMD:R_0201_0603Metric_Pad0.64x0.40mm_HandSolder
- R26: renamed from R?; footprint (none) -> Resistor_SMD:R_0201_0603Metric_Pad0.64x0.40mm_HandSolder
- SW0, SW1, TH0, TH1, TH10, TH11, TH12, TH13, TH14, TH15, TH16, TH17, TH18, TH19, TH2, TH20, TH21, TH22, TH23, TH24, TH25, TH26, TH27, TH28, TH29, TH3, TH30, TH31, TH4, TH5, TH6, TH7, TH8, TH9: footprint (none) -> Resistor_THT:R_Axial_DIN0204_L3.6mm_D1.6mm_P1.90mm_Vertical

Commit message: footprinty dokonczon, ale teraz tak na serio
Parts:
- U0: footprint MCU_RaspberryPi_and_Boards:RPi_Pico_SMD_TH -> UFC_Lib_FP:RPi_Pico_SMD_TH
Changed lines of the file:
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@@
 			)
 		)
-		(property "Footprint" "MCU_RaspberryPi_and_Boards:RPi_Pico_SMD_TH"
+		(property "Footprint" "UFC_Lib_FP:RPi_Pico_SMD_TH"
 			(at 229.87 466.09 90)
 			(effects

Commit message: pcb machen
do oceny
Parts:
- D0, D1, D2, D3, D4, D5, D6, D7, D8: footprint Diode_SMD:D_SMB_Handsoldering -> Diode_SMD:D_SMC_Handsoldering
- R6: footprint Crystal:Crystal_SMD_0603-2Pin_6.0x3.5mm_HandSoldering -> Resistor_SMD:R_0603_1608Metric_Pad0.98x0.95mm_HandSolder
- renumbered Q9 to Q0, Q0 to Q1, Q1 to Q2, Q2 to Q3, Q3 to Q4, Q4 to Q5, Q5 to Q6, Q6 to Q7, Q7 to Q8, R8 to R20, R20 to R21, R21 to R22, R22 to R23, R23 to R24, R24 to R25, R25 to R26, R26 to R27, R29 to R28
Connections:
- net ADC0: now also U0.32 (GPIO27_ADC1); no longer U0.31 (GPIO26_ADC0)
- net ADC1: now also U0.31 (GPIO26_ADC0); no longer U0.32 (GPIO27_ADC1)
- net FAN_TACHO0: now also R0.1
- net FAN_TACHO1: now also R1.1
- net FAN_TACHO2: now also R2.1
- net FAN_TACHO3: now also R3.1
- net FAN_TACHO4: now also R4.1
- net FAN_TACHO5: now also R5.1
- net FAN_TACHO6: now also R6.1
- net FAN_TACHO7: now also R7.1
- net Tacho0: now also C0.2, R0.2
- net Tacho1: now also C1.2, R1.2
- net Tacho2: now also C2.2, R2.2
- net Tacho3: now also C3.2, R3.2
- net Tacho4: now also C4.2, R4.2; no longer U0.17 (GPIO13)
- net Tacho6: now also C6.2, R6.2
- net Tacho7: now also C7.2, R7.2
- net Tacho5: now reaches C5.2, R5.2
- net Tacho5: now also U0.17 (GPIO13)

Commit message: nigger
nigger ugly ass\
Parts:
- removed U0: Pico, UFC_Lib_FP:RPi_Pico_SMD_TH, symbol MCU_RaspberryPi_and_Boards:Pico
- added PT0: ~, UFC_Lib_FP:Screw_terminal, symbol UFC_Lib:screw_terminal
- added U0: Pico_1, UFC_Lib_FP:RPi_Pico_TH, symbol UFC_Lib:Pico_1
- C0, C1, C2, C3, C4, C5, C6, C7: footprint Capacitor_THT:CP_Radial_D5.0mm_P2.00mm -> Capacitor_SMD:C_0402_1005Metric_Pad0.74x0.62mm_HandSolder
- R11, R12, R14, R15, R16, R17, R18, R27: footprint Resistor_SMD:R_0201_0603Metric_Pad0.64x0.40mm_HandSolder -> UFC_Lib_FP:F_R_0201_0603Metric_PAd0
- R13: value 470R -> 470; footprint Resistor_SMD:R_0201_0603Metric_Pad0.64x0.40mm_HandSolder -> UFC_Lib_FP:F_R_0201_0603Metric_PAd0
Connections:
- net +12V: now also PT0.1 (12V)
- net +5V: now also PT0.2 (5V)
- net ADC0: now also U0.32 (GPIO27_ADC1)
- net ADC1: now also U0.31 (GPIO26_ADC0)
- net AGND: now also U0.33 (AGND)
- net DEMUX 3.3V: now also U0.36 (3V3)
- net DEMUX(0-15)_Disable: now also U0.21 (GPIO16)
- net DEMUX(16-31)_Disable: now also U0.22 (GPIO17)
- net DEMUX-Address0: now also U0.27 (GPIO21)
- net DEMUX-Address1: now also U0.26 (GPIO20)
- net DEMUX-Address2: now also U0.25 (GPIO19)
- net DEMUX-Address3: now also U0.24 (GPIO18)
- net GND: now also PT0.3 (GND), U0.13 (GND), U0.18 (GND), U0.23 (GND), U0.28 (GND), U0.3 (GND), U0.38 (GND), U0.8 (GND)
- net PWM_NMOS0: now also U0.1 (GPIO0)
- net PWM_NMOS1: now also U0.2 (GPIO1)
- net PWM_NMOS2: now also U0.4 (GPIO2)
- net PWM_NMOS3: now also U0.5 (GPIO3)
- net PWM_NMOS4: now also U0.6 (GPIO4)
- net PWM_NMOS5: now also U0.7 (GPIO5)
- net PWM_NMOS6: now also U0.9 (GPIO6)
- net PWM_NMOS7: now also U0.10 (GPIO7)
- net Tacho0: now also U0.11 (GPIO8)
- net Tacho1: now also U0.12 (GPIO9)
- net Tacho2: now also U0.14 (GPIO10)
- net Tacho3: now also U0.15 (GPIO11)
- net Tacho4: now also U0.16 (GPIO12)
- net Tacho5: now also U0.17 (GPIO13)
- net Tacho6: now also U0.19 (GPIO14)
- net Tacho7: now also U0.20 (GPIO15)
- net Working_indicator: now also U0.29 (GPIO22)
- net at SW0.2 (B): now also U0.39 (VSYS)
Other:
- note added: "chicken jockey"

Commit message: drobny update
Parts:
- removed TH0, TH1, TH10, TH11, TH12, TH13, TH14, TH15, TH16, TH17, TH18, TH19, TH2, TH20, TH21, TH22, TH23, TH24, TH25, TH26, TH27, TH28, TH29, TH3, TH30, TH31, TH4, TH5, TH6, TH7, TH8, TH9: Thermistor_NTC, Resistor_THT:R_Axial_DIN0204_L3.6mm_D1.6mm_P1.90mm_Vertical, symbol Device:Thermistor_NTC
- added C8, C9: C, Capacitor_SMD:C_0603_1608Metric_Pad1.08x0.95mm_HandSolder, symbol Device:C
- added CONN0: ~, UFC_Lib_FP:NTC_connector_32x2, symbol UFC_Lib:ntc_connector_32x2
Connections:
- net +5V: now also C8.1, C9.1
- net ADC0: now also CONN0.17, CONN0.18, CONN0.19, CONN0.20, CONN0.21, CONN0.22, CONN0.23, CONN0.24, CONN0.25, CONN0.26, CONN0.27, CONN0.28, CONN0.29, CONN0.30, CONN0.31, CONN0.32
- net ADC1: now also CONN0.49, CONN0.50, CONN0.51, CONN0.52, CONN0.53, CONN0.54, CONN0.55, CONN0.56, CONN0.57, CONN0.58, CONN0.59, CONN0.60, CONN0.61, CONN0.62, CONN0.63, CONN0.64
- net DEMUX-Thermistor0: now also CONN0.1
- net DEMUX-Thermistor1: now also CONN0.2
- net DEMUX-Thermistor10: now also CONN0.11
- net DEMUX-Thermistor11: now also CONN0.12
- net DEMUX-Thermistor12: now also CONN0.13
- net DEMUX-Thermistor13: now also CONN0.14
- net DEMUX-Thermistor14: now also CONN0.15
- net DEMUX-Thermistor15: now also CONN0.16
- net DEMUX-Thermistor16: now also CONN0.33
- net DEMUX-Thermistor17: now also CONN0.34
- net DEMUX-Thermistor18: now also CONN0.35
- net DEMUX-Thermistor19: now also CONN0.36
- net DEMUX-Thermistor2: now also CONN0.3
- net DEMUX-Thermistor20: now also CONN0.37
- net DEMUX-Thermistor21: now also CONN0.38
- net DEMUX-Thermistor22: now also CONN0.39
- net DEMUX-Thermistor23: now also CONN0.40
- net DEMUX-Thermistor24: now also CONN0.41
- net DEMUX-Thermistor25: now also CONN0.42
- net DEMUX-Thermistor26: now also CONN0.43
- net DEMUX-Thermistor27: now also CONN0.44
- net DEMUX-Thermistor28: now also CONN0.45
- net DEMUX-Thermistor29: now also CONN0.46
- net DEMUX-Thermistor3: now also CONN0.4
- net DEMUX-Thermistor30: now also CONN0.47
- net DEMUX-Thermistor31: now also CONN0.48
- net DEMUX-Thermistor4: now also CONN0.5
- net DEMUX-Thermistor5: now also CONN0.6
- net DEMUX-Thermistor6: now also CONN0.7
- net DEMUX-Thermistor7: now also CONN0.8
- net DEMUX-Thermistor8: now also CONN0.9
- net DEMUX-Thermistor9: now also CONN0.10
- net GND: now also C8.2, C9.2
Other:
- note added: "Power terminal"
- note added: "Thermistors (0-31)"
- note removed: "Thermistors (0-15)"
- note removed: "Thermistors (16-31)"
- note removed: "chicken jockey"
- moved on the sheet: PT0, R10, R9

Commit message: nearly done
Parts:
- C0, C1, C2, C3, C4, C5, C6, C7: footprint Capacitor_SMD:C_0402_1005Metric_Pad0.74x0.62mm_HandSolder -> Capacitor_SMD:C_0603_1608Metric_Pad1.08x0.95mm_HandSolder
- C8: value C -> 1u
- R10, R9: footprint Resistor_SMD:R_0402_1005Metric_Pad0.72x0.64mm_HandSolder -> Resistor_SMD:R_0805_2012Metric_Pad1.20x1.40mm_HandSolder
- R11, R12, R14, R15, R16, R17, R18, R27: footprint UFC_Lib_FP:F_R_0201_0603Metric_PAd0 -> Resistor_SMD:R_0603_1608Metric_Pad0.98x0.95mm_HandSolder
- R13: value 470 -> 470R; footprint UFC_Lib_FP:F_R_0201_0603Metric_PAd0 -> Resistor_SMD:R_0603_1608Metric_Pad0.98x0.95mm_HandSolder
- R19, R20, R21, R22, R23, R24, R25, R26: footprint Capacitor_SMD:C_0402_1005Metric_Pad0.74x0.62mm_HandSolder -> Resistor_SMD:R_0603_1608Metric_Pad0.98x0.95mm_HandSolder
- R28: footprint Resistor_SMD:R_1206_3216Metric_Pad1.30x1.75mm_HandSolder -> Resistor_SMD:R_0603_1608Metric_Pad0.98x0.95mm_HandSolder
