File: PCB/UFC.kicad_pcb (KiCad board)
At the start: 2 copper layers, 118.5 x 89.5 mm, 101 parts, among them IC0 CD74HCT4067M, IC1 CD74HCT4067M, K0 EP1-3N1S, M0 Fan_3pin, M1 Fan_3pin, M2 Fan_3pin, M3 Fan_3pin, M4 Fan_3pin, M5 Fan_3pin, M6 Fan_3pin, M7 Fan_3pin, Q0 NMOS, Q1 NMOS, Q2 NMOS, Q3 NMOS, Q4 NMOS, Q5 NMOS, Q6 NMOS, Q7 NMOS, Q9 NMOS, SW0 MCU Reset, SW1 Main Power Switch, U0 Pico

Commit message: pcb machen
do oceny
Parts:
- D0, D1, D2, D3, D4, D5, D6, D7, D8: footprint Diode_SMD:D_SMB_Handsoldering -> Diode_SMD:D_SMC_Handsoldering
- R6: footprint Crystal:Crystal_SMD_0603-2Pin_6.0x3.5mm_HandSoldering -> Resistor_SMD:R_0603_1608Metric_Pad0.98x0.95mm_HandSolder
- SW1: moved to B.Cu
- moved R27 146.9 mm to (226.0, 88.5), turned to 90 degrees
- moved Q8 144.6 mm to (220.0, 95.0), turned to 180 degrees
- moved Q0 131.8 mm to (170.2, 61.0)
- moved Q1 129.2 mm to (170.2, 65.9)
- moved Q2 129.0 mm to (170.2, 71.0)
- moved Q3 128.7 mm to (170.2, 76.1)
- moved Q4 114.0 mm to (170.2, 81.3)
- moved Q5 113.7 mm to (170.2, 86.4)
- moved Q6 113.5 mm to (170.2, 91.5)
- moved R0 112.4 mm to (136.1, 50.8), turned to 180 degrees
- moved R1 107.2 mm to (136.1, 58.8), turned to 180 degrees
- moved R13 105.5 mm to (166.8, 72.9), turned to 90 degrees
- moved R14 103.0 mm to (166.8, 77.9), turned to 90 degrees
- moved R2 102.1 mm to (136.1, 66.8), turned to 180 degrees
- moved R15 100.2 mm to (166.8, 83.2), turned to 90 degrees
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- renumbered Q9 to Q0, Q0 to Q1, Q1 to Q2, Q2 to Q3, Q3 to Q4, Q4 to Q5, Q5 to Q6, Q6 to Q7, Q7 to Q8, R8 to R20, R20 to R21, R21 to R22, R22 to R23, R23 to R24, R24 to R25, R25 to R26, R26 to R27, R29 to R28
Connections:
- C0 pad 2: Net-(C0-Pad2) -> /Tacho0
- C1 pad 2: Net-(C1-Pad2) -> /Tacho1
- C2 pad 2: Net-(C2-Pad2) -> /Tacho2
- C3 pad 2: Net-(C3-Pad2) -> /Tacho3
- C4 pad 2: Net-(C4-Pad2) -> /Tacho4
- C5 pad 2: Net-(C5-Pad2) -> /Tacho5
- C6 pad 2: Net-(C6-Pad2) -> /Tacho6
- C7 pad 2: Net-(C7-Pad2) -> /Tacho7
- R0 pad 1: unconnected-(R0-Pad1) -> /FAN_TACHO0
- R0 pad 2: Net-(C0-Pad2) -> /Tacho0
- R1 pad 1: unconnected-(R1-Pad1) -> /FAN_TACHO1
- R1 pad 2: Net-(C1-Pad2) -> /Tacho1
- R2 pad 1: unconnected-(R2-Pad1) -> /FAN_TACHO2
- R2 pad 2: Net-(C2-Pad2) -> /Tacho2
- R3 pad 1: unconnected-(R3-Pad1) -> /FAN_TACHO3
- R3 pad 2: Net-(C3-Pad2) -> /Tacho3
- R4 pad 1: unconnected-(R4-Pad1) -> /FAN_TACHO4
- R4 pad 2: Net-(C4-Pad2) -> /Tacho4
- R5 pad 1: unconnected-(R5-Pad1) -> /FAN_TACHO5
- R5 pad 2: Net-(C5-Pad2) -> /Tacho5
- R6 pad 1: unconnected-(R6-Pad1) -> /FAN_TACHO6
- R6 pad 2: Net-(C6-Pad2) -> /Tacho6
- R7 pad 1: unconnected-(R7-Pad1) -> /FAN_TACHO7
- R7 pad 2: Net-(C7-Pad2) -> /Tacho7
- U0 pad 17: /Tacho4 -> /Tacho5
- U0 pad 31: /ADC0 -> /ADC1
- U0 pad 32: /ADC1 -> /ADC0
Routing:
- net +12V: track 0.00 -> 134.3 mm
- net /Tacho1: track 0.00 -> 107.6 mm
- net /Tacho2: track 0.00 -> 106.3 mm, vias 0 -> 2
- net /Tacho0: track 0.00 -> 103.9 mm
- net /Tacho3: track 0.00 -> 88.0 mm
- net /Relay_closed: track 0.00 -> 82.9 mm
- net /ADC0: track 0.00 -> 82.2 mm, vias 0 -> 3
- net /DEMUX-Address2: track 0.00 -> 81.2 mm, vias 0 -> 2
- net /Tacho4: track 0.00 -> 81.2 mm
- net /DEMUX 3.3V: track 0.00 -> 80.8 mm, vias 0 -> 3
- net /ADC1: track 0.00 -> 80.1 mm, vias 0 -> 2
- net /DEMUX-Address0: track 0.00 -> 77.9 mm, vias 0 -> 2
- net /DEMUX-Address1: track 0.00 -> 73.4 mm, vias 0 -> 2
- net Net-(D8-A): track 0.00 -> 72.5 mm
- net /DEMUX-Address3: track 0.00 -> 71.0 mm, vias 0 -> 2
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Other:
- board outline removed

Commit message: nigger
nigger ugly ass\
Parts:
- added PT0: ~, UFC_Lib_FP:Screw_terminal, F.Cu at (173.5, 108.0)
- C0, C1, C2, C3, C4, C5, C6, C7: footprint Capacitor_THT:CP_Radial_D5.0mm_P2.00mm -> Capacitor_SMD:C_0402_1005Metric_Pad0.74x0.62mm_HandSolder
- R11, R12, R14, R15, R16, R17, R18, R27: footprint Resistor_SMD:R_0201_0603Metric_Pad0.64x0.40mm_HandSolder -> UFC_Lib_FP:F_R_0201_0603Metric_PAd0
- R13: value 470R -> 470; footprint Resistor_SMD:R_0201_0603Metric_Pad0.64x0.40mm_HandSolder -> UFC_Lib_FP:F_R_0201_0603Metric_PAd0
- U0: value Pico -> Pico_1; footprint UFC_Lib_FP:RPi_Pico_SMD_TH -> UFC_Lib_FP:RPi_Pico_TH
- moved TH0 19.5 mm to (222.5, 52.9), turned to 90 degrees
- moved TH16 18.0 mm to (242.5, 52.9), turned to 90 degrees
- moved TH2 16.9 mm to (225.0, 52.9), turned to 90 degrees
- moved TH14 15.6 mm to (240.0, 52.9), turned to 90 degrees
- moved TH4 14.7 mm to (227.5, 52.9), turned to 90 degrees
- moved TH18 14.4 mm to (241.1, 59.0)
- moved TH20 14.4 mm to (241.1, 61.5)
- moved TH22 14.4 mm to (241.1, 64.0)
- moved TH24 14.4 mm to (241.1, 66.5)
- moved TH26 14.4 mm to (241.1, 69.0)
- moved TH28 14.4 mm to (241.1, 71.5)
- moved TH30 14.4 mm to (241.1, 74.0)
- moved TH12 13.8 mm to (237.5, 52.9), turned to 90 degrees
- moved TH1 13.2 mm to (241.1, 79.0)
- moved TH11 13.2 mm to (241.1, 91.5)
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Routing:
- net +5V: track 66.3 -> 125.9 mm, vias 3 -> 5
- net +12V: track 134.3 -> 158.6 mm
- net GND: track 3.40 -> 20.7 mm, vias 0 -> 181
- net /DEMUX-Address2: track 81.2 -> 67.1 mm
- net /DEMUX-Thermistor8: track 12.7 -> 26.2 mm
- net /DEMUX-Thermistor9: track 13.2 -> 25.4 mm
- net /ADC0: track 82.2 -> 92.9 mm
- net /DEMUX-Thermistor0: track 24.2 -> 13.7 mm
- net /DEMUX-Thermistor10: track 14.1 -> 24.2 mm
- net /DEMUX-Thermistor11: track 15.1 -> 23.6 mm
- net /DEMUX-Thermistor1: track 21.9 -> 13.5 mm
- net /DEMUX-Address3: track 71.0 -> 63.0 mm, vias 2 -> 3
- net /DEMUX-Thermistor2: track 19.6 -> 12.4 mm
- net /Tacho0: track 103.9 -> 96.7 mm, vias 0 -> 1
- net /DEMUX-Thermistor16: track 24.2 -> 31.0 mm
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- added copper zone on B.Cu, net +12V
- added copper zone on B.Cu, net GND
- added copper zone on F.Cu, net GND
Other:
- board outline added: 117.5 x 75 mm

Commit message: drobny update
Parts:
- removed TH0, TH1, TH10, TH11, TH12, TH13, TH14, TH15, TH16, TH17, TH18, TH19, TH2, TH20, TH21, TH22, TH23, TH24, TH25, TH26, TH27, TH28, TH29, TH3, TH30, TH31, TH4, TH5, TH6, TH7, TH8, TH9: Thermistor_NTC, Resistor_THT:R_Axial_DIN0204_L3.6mm_D1.6mm_P1.90mm_Vertical
- added C8: C, Capacitor_SMD:C_0603_1608Metric_Pad1.08x0.95mm_HandSolder, F.Cu at (149.1, 110.0)
- added C9: C, Capacitor_SMD:C_0603_1608Metric_Pad1.08x0.95mm_HandSolder, F.Cu at (149.1, 112.5)
- added CONN0: ~, UFC_Lib_FP:NTC_connector_32x2, F.Cu at (233.7, 64.8)
- SW1: moved to F.Cu
- moved D8 122.0 mm to (106.6, 112.2)
- moved F0 97.4 mm to (141.0, 124.7), turned to 0 degrees
- moved SW0 93.4 mm to (156.3, 123.8), turned to 0 degrees
- moved Q8 91.3 mm to (130.2, 111.5), turned to 0 degrees
- moved SW1 75.8 mm to (156.3, 127.0), turned to 0 degrees
- moved U0 71.9 mm to (126.1, 70.9)
- moved R27 69.1 mm to (164.5, 120.0), turned to 0 degrees
- moved K0 68.7 mm to (140.6, 97.7), turned to 0 degrees
- moved Q0 67.0 mm to (117.3, 101.9)
- moved Q1 66.9 mm to (117.3, 106.7)
- moved Q2 66.7 mm to (117.3, 111.5)
- moved R9 64.3 mm to (161.3, 123.3)
- moved R28 64.0 mm to (157.8, 99.3), turned to 0 degrees
- moved R10 60.8 mm to (161.3, 125.3), turned to 0 degrees
- moved Q3 53.2 mm to (123.7, 101.9)
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Routing:
- net +12V: track 158.6 -> 0.00 mm
- net +5V: track 125.9 -> 0.00 mm, vias 5 -> 0
- net /Tacho1: track 101.9 -> 0.00 mm, vias 1 -> 0
- net /Tacho2: track 101.3 -> 0.00 mm, vias 3 -> 0
- net /Tacho0: track 96.7 -> 0.00 mm, vias 1 -> 0
- net /ADC0: track 92.9 -> 0.00 mm, vias 3 -> 0
- net /ADC1: track 86.4 -> 0.00 mm, vias 2 -> 0
- net /Tacho3: track 85.5 -> 0.00 mm, vias 1 -> 0
- net /Relay_closed: track 82.9 -> 0.00 mm
- net /Tacho4: track 79.1 -> 0.00 mm, vias 1 -> 0
- net /DEMUX 3.3V: track 76.4 -> 0.00 mm, vias 3 -> 0
- net /DEMUX-Address1: track 74.2 -> 0.00 mm, vias 2 -> 0
- net /DEMUX-Address0: track 74.1 -> 0.00 mm, vias 2 -> 0
- net /Tacho5: track 72.4 -> 0.00 mm, vias 1 -> 0
- net Net-(D8-A): track 71.2 -> 0.00 mm
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- removed copper zone on B.Cu, net +12V
- removed copper zone on B.Cu, net GND
- removed copper zone on F.Cu, net GND
Other:
- board outline removed

Commit message: nearly done
Parts:
- C0, C1, C2, C3, C4, C5, C6, C7: footprint Capacitor_SMD:C_0402_1005Metric_Pad0.74x0.62mm_HandSolder -> Capacitor_SMD:C_0603_1608Metric_Pad1.08x0.95mm_HandSolder; moved to B.Cu
- C8: value C -> 1u
- D0, D1, D2, D3, D4, D5, D6, D7, D8, Q0, Q1, Q2, Q3, Q4, Q5, Q6, Q7, Q8, R0, R1, R2, R3, R4, R5, R6, R7, SW1: moved to B.Cu
- R10, R9: footprint Resistor_SMD:R_0402_1005Metric_Pad0.72x0.64mm_HandSolder -> Resistor_SMD:R_0805_2012Metric_Pad1.20x1.40mm_HandSolder; moved to B.Cu
- R11, R12, R14, R15, R16, R17, R27: footprint UFC_Lib_FP:F_R_0201_0603Metric_PAd0 -> Resistor_SMD:R_0603_1608Metric_Pad0.98x0.95mm_HandSolder; moved to B.Cu
- R13: value 470 -> 470R; footprint UFC_Lib_FP:F_R_0201_0603Metric_PAd0 -> Resistor_SMD:R_0603_1608Metric_Pad0.98x0.95mm_HandSolder; moved to B.Cu
- R18: footprint UFC_Lib_FP:F_R_0201_0603Metric_PAd0 -> Resistor_SMD:R_0603_1608Metric_Pad0.98x0.95mm_HandSolder
- R19, R20, R21, R22, R23, R24, R25, R26: footprint Capacitor_SMD:C_0402_1005Metric_Pad0.74x0.62mm_HandSolder -> Resistor_SMD:R_0603_1608Metric_Pad0.98x0.95mm_HandSolder; moved to B.Cu
- R28: footprint Resistor_SMD:R_1206_3216Metric_Pad1.30x1.75mm_HandSolder -> Resistor_SMD:R_0603_1608Metric_Pad0.98x0.95mm_HandSolder; moved to B.Cu
- moved D8 129.5 mm to (236.0, 107.2), turned to 90 degrees
- moved F0 107.3 mm to (246.4, 144.3)
- moved Q8 106.0 mm to (235.1, 96.0), turned to 90 degrees
- moved PT0 104.7 mm to (225.8, 143.9)
- moved C8 96.9 mm to (243.0, 85.7)
- moved C9 94.8 mm to (243.0, 125.7)
- moved R6 90.4 mm to (201.9, 142.0), turned to 90 degrees
- moved R9 88.7 mm to (234.2, 72.9), turned to 90 degrees
- moved U0 87.9 mm to (212.1, 89.0)
- moved R10 86.8 mm to (235.2, 79.8)
- moved K0 84.8 mm to (221.4, 123.2), turned to 180 degrees
- moved R7 83.9 mm to (195.9, 140.3), turned to 90 degrees
- moved Q0 82.9 mm to (190.4, 62.9)
- moved SW0 81.7 mm to (224.8, 79.3), turned to 90 degrees
- moved SW1 81.6 mm to (231.0, 94.1), turned to -90 degrees
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Routing:
- net +12V: track 0.00 -> 208.0 mm
- net /Relay_closed: track 0.00 -> 133.9 mm
- net /FAN_TACHO4: track 0.00 -> 115.8 mm
- net +5V: track 0.00 -> 109.4 mm, vias 0 -> 2
- net /Relay_open: track 0.00 -> 106.6 mm
- net /ADC1: track 0.00 -> 106.0 mm
- net /FAN_TACHO5: track 0.00 -> 105.4 mm, vias 0 -> 2
- net /FAN_TACHO3: track 0.00 -> 96.2 mm
- net /ADC0: track 0.00 -> 82.5 mm
- net /FAN_TACHO2: track 0.00 -> 66.6 mm
- net /DEMUX 3.3V: track 0.00 -> 65.4 mm, vias 0 -> 2
- net /DEMUX-Address0: track 0.00 -> 62.9 mm, vias 0 -> 1
- net /DEMUX-Address3: track 0.00 -> 60.2 mm, vias 0 -> 1
- net /FAN_TACHO1: track 0.00 -> 59.4 mm
- net /FAN_TACHO0: track 0.00 -> 58.1 mm
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- added copper zone on B.Cu, net GND
- added copper zone on F.Cu, net GND
Other:
- board outline added: 98 x 100 mm

Commit message: pcb update
finished probably
Parts:
- R18: moved to B.Cu
- SW1: moved to F.Cu
Routing:
- net Net-(Q7-G): vias 1 -> 2
- net GND: vias 0 -> 248
Other:
- board size 98 x 100 mm -> 100 x 100 mm

Commit message: 1
Routing:
- net GND: vias 248 -> 267
Changed lines of the file:
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@@
+	)
+	(via
+		(at 258 141)
+		(size 0.6)
+		(drill 0.3)
+		(layers "F.Cu" "B.Cu")
+		(free yes)
+		(net 1)
 	)
 	(via
@@
 	)
 	(via
+		(at 252 141)
+		(size 0.6)
+		(drill 0.3)
+		(layers "F.Cu" "B.Cu")
+		(free yes)
+		(net 1)
+	)
+	(via
 		(at 223.5 68)
 		(size 0.6)
@@
 	)
 	(via
+		(at 253.5 141)
+		(size 0.6)
+		(drill 0.3)
+		(layers "F.Cu" "B.Cu")
+		(free yes)
+		(net 1)
+	)
+	(via
 		(at 256.8 100.2)
 		(size 0.6)
@@
 	)
 	(via
+		(at 259.5 141)
+		(size 0.6)
+		(drill 0.3)
+		(layers "F.Cu" "B.Cu")
+		(free yes)
+		(net 1)
+	)
+	(via
 		(at 227 149)
 		(size 0.6)
@@
 	)
 	(via
+		(at 256.5 141)
+		(size 0.6)
+		(drill 0.3)
+		(layers "F.Cu" "B.Cu")
+		(free yes)
+		(net 1)
+	)
+	(via
 		(at 231.5 109)
 		(size 0.6)
@@
 	)
 	(via
+		(at 251 145)
+		(size 0.6)
+		(drill 0.3)
+		(layers "F.Cu" "B.Cu")
+		(free yes)
+		(net 1)
+	)
+	(via
+		(at 261 141)
+		(size 0.6)
+		(drill 0.3)
+		(layers "F.Cu" "B.Cu")
+		(free yes)
+		(net 1)
+	)
+	(via
 		(at 231 89.5)
 		(size 0.6)
@@
 	)
 	(via
+		(at 235.55 106.32)
+		(size 0.6)
+		(drill 0.3)
+		(layers "F.Cu" "B.Cu")
+		(free yes)
+		(net 1)
+	)
+	(via
 		(at 247.5 85.5)
 		(size 0.6)
@@
 	)
 	(via
+		(at 251 143.5)
+		(size 0.6)
+		(drill 0.3)
+		(layers "F.Cu" "B.Cu")
+		(free yes)
+		(net 1)
+	)
+	(via
 		(at 219 77)
 		(size 0.6)
@@
 	)
 	(via
+		(at 255 141)
+		(size 0.6)
+		(drill 0.3)
+		(layers "F.Cu" "B.Cu")
+		(free yes)
+		(net 1)
+	)
+	(via
 		(at 261 149.5)
 		(size 0.6)
@@
 	)
 	(via
+		(at 238.29 98.23)
+		(size 0.6)
+		(drill 0.3)
+		(layers "F.Cu" "B.Cu")
+		(free yes)
+		(net 1)
+	)
+	(via
 		(at 200.5 107.5)
 		(size 0.6)
@@
 	)
 	(via
+		(at 234.53 107.35)
+		(size 0.6)
+		(drill 0.3)
+		(layers "F.Cu" "B.Cu")
+		(free yes)
+		(net 1)
+	)
+	(via
 		(at 229.5 103.5)
 		(size 0.6)
@@
 	)
 	(via
+		(at 251 149.5)
+		(size 0.6)
+		(drill 0.3)
+		(layers "F.Cu" "B.Cu")
+		(free yes)
+		(net 1)
+	)
+	(via
 		(at 233.5 102)
 		(size 0.6)
@@
 	)
 	(via
+		(at 251 141)
+		(size 0.6)
+		(drill 0.3)
+		(layers "F.Cu" "B.Cu")
+		(free yes)
+		(net 1)
+	)
+	(via
 		(at 201.5 86)
 		(size 0.6)
@@
 	)
 	(via
+		(at 251 142)
+		(size 0.6)
+		(drill 0.3)
+		(layers "F.Cu" "B.Cu")
+		(free yes)
+		(net 1)
+	)
+	(via
 		(at 253.5 142)
 		(size 0.6)
@@
 	)
 	(via
+		(at 251 151)
+		(size 0.6)
+		(drill 0.3)
+		(layers "F.Cu" "B.Cu")
+		(free yes)
+		(net 1)
+	)
+	(via
 		(at 198.5 111.5)
 		(size 0.6)
@@
 	)
 	(via
+		(at 238.33 96.54)
+		(size 0.6)
+		(drill 0.3)
+		(layers "F.Cu" "B.Cu")
+		(free yes)
+		(net 1)
+	)
+	(via
 		(at 245.5 83.5)
 		(size 0.6)
@@
 	)
 	(via
+		(at 251 146.5)
+		(size 0.6)
+		(drill 0.3)
+		(layers "F.Cu" "B.Cu")
+		(free yes)
+		(net 1)
+	)
+	(via
 		(at 219 88)
 		(size 0.6)
@@
 	(via
 		(at 233.5 100.5)
+		(size 0.6)
+		(drill 0.3)
+		(layers "F.Cu" "B.Cu")
+		(free yes)
+		(net 1)
+	)
+	(via
+		(at 251 148)
 		(size 0.6)
 		(drill 0.3)
@@
 	(segment
 		(start 175.201 142.975066)
-		(end 179.924934 147.699)
+		(end 176.112967 143.887033)
 		(width 5.5)
 		(layer "B.Cu")
@@
 	)
 	(segment
-		(start 179.924934 147.699)
+		(start 181.996002 147.699)
 		(end 205.301 147.699)
 		(width 5.5)
@@
 	)
 	(segment
+		(start 176.112967 143.887033)
+		(end 178.460468 146.234534)
+		(width 5.5)
+		(layer "B.Cu")
+		(net 3)
+	)
+	(segment
 		(start 175.201 77.8)
 		(end 175.201 142.975066)
 		(width 5.5)
 		(layer "B.Cu")
+		(net 3)
+	)
+	(arc
+		(start 178.460468 146.234534)
+		(mid 180.082585 147.318398)
+		(end 181.996002 147.699)
+		(width 5.5)
+		(layer "B.Cu")

Commit message: f
Routing:
- net GND: vias 267 -> 355
