File: PCB/UFC.kicad_pcb (KiCad board)
At the start: 2 copper layers, 100 x 100 mm, 73 parts, among them IC0 CD74HCT4067M, IC1 CD74HCT4067M, K0 EP1-3N1S, M0 Fan_3pin, M1 Fan_3pin, M2 Fan_3pin, M3 Fan_3pin, M4 Fan_3pin, M5 Fan_3pin, M6 Fan_3pin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

Commit message: silkscreen machen
Parts:
- added G***: LOGO, LOGO, F.Cu at (176.0, 77.0)
- added G***: LOGO, LOGO, F.Cu at (242.4, 100.1)
Other:
- board text added: "Bartosz Nocoń"
- board text added: "microsystem oriented society"

Commit message: wiecej oznaczen
Parts:
- moved G*** 3.47 mm to (240.6, 103.1)
- moved CONN0 0.05 mm to (258.7, 90.9)
Connections:
- M0 pad : /NMOS-FAN0 -> (no net)
- M1 pad : /NMOS-FAN1 -> (no net)
- M2 pad : /NMOS-FAN2 -> (no net)
- M3 pad : /NMOS-FAN3 -> (no net)
- M4 pad : /NMOS-FAN4 -> (no net)
- M5 pad : /NMOS-FAN5 -> (no net)
- M6 pad : /NMOS-FAN6 -> (no net)
- M7 pad : /NMOS-FAN7 -> (no net)
Routing:
- net /DEMUX-Thermistor31: track 29.0 -> 29.9 mm
- net GND: vias 355 -> 352
Other:
- outline, holes or cut-outs redrawn
